Commit message: oppsies

File: src/arm_description_pkg/urdf/robotic_arm.urdf (robot description, URDF)
Before this commit: robot six-axis, 10 links, 9 joints
Links:
- removed link l0
- removed link l1
- removed link l2
- removed link l3
- removed link l4
- removed link l5
- removed link l6
- removed link le
- removed link le_1
- added link gripper_center
- added link link_bicep; collision box size=0.03 0.04 0.105; visual box size=0.03 0.04 0.105
- added link link_forearm; collision box size=0.025 0.035 0.145; visual box size=0.025 0.035 0.145
- added link link_gripper_base; collision box size=0.04 0.06 0.047; visual box size=0.04 0.06 0.047
- added link link_gripper_left_finger; collision box size=0.01 0.01 0.06; visual box size=0.01 0.01 0.06
- added link link_gripper_right_finger; collision box size=0.01 0.01 0.06; visual box size=0.01 0.01 0.06
- added link link_shoulder; collision cylinder length=0.015 radius=0.04; visual cylinder length=0.015 radius=0.04
- added link link_wrist_roll; collision cylinder length=0.075 radius=0.02; visual cylinder length=0.075 radius=0.02
- link base_link: geometry collision cylinder length=0.126 radius=0.06; visual cylinder length=0.126 radius=0.06
Joints:
- removed joint j0
- removed joint j1
- removed joint j2
- removed joint j3
- removed joint j4
- removed joint j5
- removed joint j6
- removed joint j_dummy
- removed joint j_dummy_1_2
- added joint joint_1_gripper: type revolute, parent link_gripper_base, child link_gripper_left_finger, origin xyz=0 0.015 0.047 rpy=-0.5236 0 0, axis 1 0 0, limit lower=-0.3491 upper=0.6981 effort=10.0 velocity=1.0
- added joint joint_1_gripper_right: type revolute, parent link_gripper_base, child link_gripper_right_finger, origin xyz=0 -0.015 0.047 rpy=0.5236 0 0, axis 1 0 0, limit lower=-0.6981 upper=0.3491 effort=10.0 velocity=1.0, mimic joint=joint_1_gripper multiplier=-1.0
- added joint joint_2_wrist_roll: type revolute, parent link_wrist_roll, child link_gripper_base, origin xyz=0 0 0.075 rpy=0 0 0, axis 0 0 1, limit lower=-1.3963 upper=1.3963 effort=10.0 velocity=1.0
- added joint joint_3_wrist_pitch: type revolute, parent link_forearm, child link_wrist_roll, origin xyz=0 0 0.145 rpy=0 0 0, axis 0 1 0, limit lower=-1.5708 upper=1.5708 effort=10.0 velocity=1.0
- added joint joint_4_elbow: type revolute, parent link_bicep, child link_forearm, origin xyz=0 0 0.105 rpy=0 0 0, axis 0 -1 0, limit lower=-1.3963 upper=1.3963 effort=10.0 velocity=1.0
- added joint joint_5_shoulder: type revolute, parent link_shoulder, child link_bicep, origin xyz=0 0 0.015 rpy=0 0 0, axis 0 -1 0, limit lower=-1.2217 upper=1.2217 effort=10.0 velocity=1.0
- added joint joint_6_base: type revolute, parent base_link, child link_shoulder, origin xyz=0 0 0.126 rpy=0 0 0, axis 0 0 1, limit lower=-1.5708 upper=1.5708 effort=10.0 velocity=1.0
- added joint joint_tcp: type fixed, parent link_gripper_base, child gripper_center, origin xyz=0 0 0.107 rpy=0 0 0
