Commit message: some day the arm will do the ik

File: src/arm_description_pkg/urdf/idk_arm.urdf (robot description, URDF)
Before this commit: robot custom_6dof_arm_final, 7 links, 6 joints
Links:
- added link tool0; visual sphere radius=0.008
- link base_link: geometry collision cylinder length=0.1268 radius=0.06; visual cylinder length=0.1268 radius=0.06
- link link_bicep: geometry collision box size=0.03 0.04 0.1053; visual box size=0.03 0.04 0.1053
- link link_forearm: geometry collision box size=0.025 0.035 0.1463; visual box size=0.025 0.035 0.1463
- link link_shoulder: geometry collision cylinder length=0.0152 radius=0.04; visual cylinder length=0.0152 radius=0.04
- link link_wrist_roll: geometry collision cylinder length=0.0747 radius=0.02; visual cylinder length=0.0747 radius=0.02
Joints:
- added joint tool0_fixed_joint: type fixed, parent link_gripper_base, child tool0, origin xyz=0 0 0.1047 rpy=0 0 0
- joint joint_2_wrist_roll: origin xyz=0 0 0.075 -> xyz=0 0 0.0747
- joint joint_3_wrist_pitch: origin xyz=0 0 0.145 -> xyz=0 0 0.1463
- joint joint_4_elbow: origin xyz=0 0 0.105 -> xyz=0 0 0.1053
- joint joint_5_shoulder: origin xyz=0 0 0.015 -> xyz=0 0 0.0152
- joint joint_6_base: origin xyz=0 0 0.126 -> xyz=0 0 0.1268

Commit message: finally lets start with the MAS.

File: src/arm_description_pkg/urdf/idk_arm.urdf (robot description, URDF)
Before this commit: robot custom_6dof_arm_final, 8 links, 7 joints
Links:
- link base_link: geometry collision cylinder length=0.1010 radius=0.06; visual cylinder length=0.1010 radius=0.06
- link link_bicep: geometry collision box size=0.03 0.04 0.1041; visual box size=0.03 0.04 0.1041
- link link_wrist_roll: geometry collision cylinder length=0.0732 radius=0.02; visual cylinder length=0.0732 radius=0.02
Joints:
- joint joint_2_wrist_roll: origin xyz=0 0 0.0747 -> xyz=0 0 0.0732
- joint joint_4_elbow: origin xyz=0 0 0.1053 -> xyz=0 0 0.1041
- joint joint_6_base: origin xyz=0 0 0.1268 -> xyz=0 0 0.1010
- joint tool0_fixed_joint: origin xyz=0 0 0.1047 rpy=0 0 0 -> xyz=0 0.0132 0.1047 rpy=0 0 0
